File: Hardware/KiCad/altimeter.kicad_pcb (KiCad board)
At the start: 2 copper layers, 44 parts, among them P1 CONN_01X04, P2 CONN_01X04, P3 CONN_01X01, P4 CONN_01X01, Q1 DMN2008LFU, Q2 DMN2008LFU, Q3 DMN2008LFU, Q4 DMN2008LFU, SW1 SPST, U1 SAMD21G18A-AUT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

Commit message: board connected
Parts:
- C6, D2, P1, P2, SP1, SW1, U3: moved to B.Cu
- moved C12 140.6 mm to (128.7, 62.0), turned to 270 degrees
- moved C11 136.7 mm to (128.7, 58.6), turned to 90 degrees
- moved C13 133.9 mm to (134.4, 67.2), turned to 270 degrees
- moved C2 133.1 mm to (143.6, 52.4), turned to 180 degrees
- moved U5 131.9 mm to (133.1, 60.0), turned to 270 degrees
- moved C15 131.5 mm to (133.2, 64.2), turned to 180 degrees
- moved C17 130.2 mm to (136.3, 67.2), turned to 90 degrees
- moved C16 123.3 mm to (138.0, 63.5)
- moved U4 122.1 mm to (139.6, 66.9), turned to 90 degrees
- moved C14 121.5 mm to (138.6, 60.5), turned to 90 degrees
- moved L1 120.2 mm to (156.0, 52.9), turned to 90 degrees
- moved C4 119.6 mm to (153.9, 52.9), turned to 270 degrees
- moved P4 117.0 mm to (129.3, 53.1)
- moved U7 115.7 mm to (136.8, 53.9), turned to 90 degrees
- moved R6 114.9 mm to (150.5, 53.1), turned to 270 degrees
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Routing:
- net GND: track 0.00 -> 220.3 mm, vias 0 -> 4
- net +3V3: track 0.00 -> 156.1 mm, vias 0 -> 6
- net /SCL: track 0.00 -> 75.7 mm, vias 0 -> 6
- net Net-(D2-Pad2): track 0.00 -> 65.5 mm, vias 0 -> 1
- net /D2: track 0.00 -> 55.8 mm, vias 0 -> 3
- net /A1: track 0.00 -> 53.9 mm, vias 0 -> 2
- net /D3: track 0.00 -> 50.6 mm, vias 0 -> 2
- net /D4: track 0.00 -> 49.1 mm, vias 0 -> 2
- net /SDA: track 0.00 -> 44.7 mm, vias 0 -> 3
- net /A2: track 0.00 -> 42.8 mm, vias 0 -> 2
- net Net-(D1-Pad2): track 0.00 -> 41.0 mm, vias 0 -> 1
- net /D6: track 0.00 -> 34.8 mm, vias 0 -> 2
- net +5V: track 0.00 -> 34.8 mm, vias 0 -> 1
- net Net-(Q2-Pad1): track 0.00 -> 33.2 mm, vias 0 -> 2
- net /A4: track 0.00 -> 30.8 mm, vias 0 -> 2
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Other:
- board outline added: 50.8 x 19 mm
- net class Default: clearance 0.2 -> 0.2032; trace_width 0.25 -> 0.2032; via_dia 0.6 -> 0.7112; via_drill 0.4 -> 0.3556
- net class battery added: clearance 0.2032, trace_width 0.508, via_dia 0.7112, via_drill 0.3556
- net class power added: clearance 0.2032, trace_width 0.2794, via_dia 0.7112, via_drill 0.3556
- net class pyro added: clearance 0.2032, trace_width 1.27, via_dia 0.7112, via_drill 0.3556
- rule trace_clearance: 0.2 -> 0.2032

Commit message: Board v0.1 ordered
Routing:
- added copper zone on B.Cu, net GND
- added copper zone on F.Cu, net GND
Other:
- board text added: "v0.1"
Changed lines of the file:
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@@
     (links 145)
     (no_connects 0)
-    (area 126.924999 50.724999 177.875001 69.925001)
+    (area 126.1718 47.556257 178.6038 77.258)
     (thickness 1.6)
-    (drawings 4)
+    (drawings 5)
     (tracks 840)
     (zones 0)
@@
   )
   (setup
-    (last_trace_width 0.2794)
+    (last_trace_width 0.2032)
     (user_trace_width 0.2032)
     (user_trace_width 0.254)
@@
     (user_trace_width 1.27)
     (trace_clearance 0.2032)
-    (zone_clearance 0.508)
+    (zone_clearance 0.1524)
     (zone_45_only no)
     (trace_min 0.2)
@@
     (visible_elements 7FFEFFFF)
     (pcbplotparams
-      (layerselection 0x00030_80000001)
+      (layerselection 0x0100c_00000000)
       (usegerberextensions false)
       (excludeedgelayer true)
@@
       (outputformat 1)
       (mirror false)
-      (drillshape 1)
+      (drillshape 0)
       (scaleselection 1)
-      (outputdirectory ""))
+      (outputdirectory stencil_gerber/))
   )
   (net 0 "")
@@
     (uvia_drill 0.1016)
   )
+  (module altimeterComponentFootprints:1pin (layer F.Cu)
+    (at 159.15 67.4)
+    (descr "module 1 pin (ou trou mecanique de percage)")
+    (tags DEV)
+    (fp_text reference P3 (at 0.1 -0.25) (layer F.SilkS)
+      (effects (font (size 1 1) (thickness 0.15)))
+    )
+    (fp_text value CONN_01X01 (at 0 3.3528) (layer F.Fab)
+      (effects (font (size 1 1) (thickness 0.15)))
+    )
+    (fp_circle (center 0 0) (end 0 -2.286) (layer F.SilkS) (width 0.15))
+    (pad 1 thru_hole circle (at 0 0) (size 3.375 3.375) (drill 2.325) (layers *.Cu *.Mask F.SilkS))
+  )
+  (module altimeterComponentFootprints:1pin (layer F.Cu)
+    (at 129.35 53.15)
+    (descr "module 1 pin (ou trou mecanique de percage)")
+    (tags DEV)
+    (fp_text reference P4 (at 0 -0.1) (layer F.SilkS)
+      (effects (font (size 1 1) (thickness 0.15)))
+    )
+    (fp_text value CONN_01X01 (at 0 3.3528) (layer F.Fab)
+      (effects (font (size 1 1) (thickness 0.15)))
+    )
+    (fp_circle (center 0 0) (end 0 -2.286) (layer F.SilkS) (width 0.15))
+    (pad 1 thru_hole circle (at 0 0) (size 3.375 3.375) (drill 2.325) (layers *.Cu *.Mask F.SilkS))
+  )
+  (module altimeterComponentFootprints:PB-5R0H104-R_Super_Capacitor_horizontal (layer B.Cu)
+    (at 159.05 66.25 180)
+    (fp_text reference C6 (at 0.8 7.7 180) (layer B.SilkS)
+      (effects (font (size 1 1) (thickness 0.15)) (justify mirror))
+    )
+    (fp_text value 100mF (at -0.0254 -2.0574 180) (layer B.Fab)
+      (effects (font (size 1 1) (thickness 0.15)) (justify mirror))
+    )
+    (fp_line (start -5.65 2) (end -5.65 15) (layer B.SilkS) (width 0.15))
+    (fp_line (start -5.65 15) (end 5.65 15) (layer B.SilkS) (width 0.15))
+    (fp_line (start 5.65 15) (end 5.65 2) (layer B.SilkS) (width 0.15))
+    (fp_line (start 5.65 2) (end -5.65 2) (layer B.SilkS) (width 0.15))
+    (fp_line (start -3.6576 0.7112) (end -3.6576 1.4478) (layer B.SilkS) (width 0.15))
+    (fp_line (start -4.0386 1.0668) (end -3.302 1.0668) (layer B.SilkS) (width 0.15))
+    (pad 1 thru_hole circle (at -3.65 0 180) (size 1.01 1.01) (drill 0.65) (layers *.Cu *.Mask)
+      (net 7 "Net-(C6-Pad1)"))
+    (pad 2 thru_hole circle (at 3.65 0 180) (size 1.01 1.01) (drill 0.65) (layers *.Cu *.Mask)
+      (net 1 GND))
+  )
   (module altimeterComponentFootprints:TQFP-48_7x7mm_Pitch0.5mm (layer F.Cu)
     (at 146.7 60.5 225)
@@
     )
   )
-  (module altimeterComponentFootprints:PB-5R0H104-R_Super_Capacitor_horizontal (layer B.Cu)
-    (at 159.05 66.25 180)
-    (fp_text reference C6 (at 0.8 7.7 180) (layer B.SilkS)
-      (effects (font (size 1 1) (thickness 0.15)) (justify mirror))
-    )
-    (fp_text value 100mF (at -0.0254 -2.0574 180) (layer B.Fab)
-      (effects (font (size 1 1) (thickness 0.15)) (justify mirror))
-    )
-    (fp_line (start -5.65 2) (end -5.65 15) (layer B.SilkS) (width 0.15))
-    (fp_line (start -5.65 15) (end 5.65 15) (layer B.SilkS) (width 0.15))
-    (fp_line (start 5.65 15) (end 5.65 2) (layer B.SilkS) (width 0.15))
-    (fp_line (start 5.65 2) (end -5.65 2) (layer B.SilkS) (width 0.15))
-    (fp_line (start -3.6576 0.7112) (end -3.6576 1.4478) (layer B.SilkS) (width 0.15))
-    (fp_line (start -4.0386 1.0668) (end -3.302 1.0668) (layer B.SilkS) (width 0.15))
-    (pad 1 thru_hole circle (at -3.65 0 180) (size 1.01 1.01) (drill 0.65) (layers *.Cu *.Mask)
-      (net 7 "Net-(C6-Pad1)"))
-    (pad 2 thru_hole circle (at 3.65 0 180) (size 1.01 1.01) (drill 0.65) (layers *.Cu *.Mask)
-      (net 1 GND))
-  )
   (module altimeterComponentFootprints:C_0603 (layer F.Cu)
     (at 151.95 65.55 180)
@@
     (pad 4 thru_hole rect (at 3.81 0 180) (size 1.52 1.52) (drill 1.01) (layers *.Cu *.Mask)
       (net 1 GND))
-  )
-  (module altimeterComponentFootprints:1pin (layer F.Cu)
-    (at 159.15 67.4)
-    (descr "module 1 pin (ou trou mecanique de percage)")
-    (tags DEV)
-    (fp_text reference P3 (at 0.1 -0.25) (layer F.SilkS)
-      (effects (font (size 1 1) (thickness 0.15)))
-    )
-    (fp_text value CONN_01X01 (at 0 3.3528) (layer F.Fab)
-      (effects (font (size 1 1) (thickness 0.15)))
-    )
-    (fp_circle (center 0 0) (end 0 -2.286) (layer F.SilkS) (width 0.15))
-    (pad 1 thru_hole circle (at 0 0) (size 3.375 3.375) (drill 2.325) (layers *.Cu *.Mask F.SilkS))
-  )
-  (module altimeterComponentFootprints:1pin (layer F.Cu)
-    (at 129.35 53.15)
-    (descr "module 1 pin (ou trou mecanique de percage)")
-    (tags DEV)
-    (fp_text reference P4 (at 0 -0.1) (layer F.SilkS)
-      (effects (font (size 1 1) (thickness 0.15)))
-    )
-    (fp_text value CONN_01X01 (at 0 3.3528) (layer F.Fab)
-      (effects (font (size 1 1) (thickness 0.15)))
-    )
-    (fp_circle (center 0 0) (end 0 -2.286) (layer F.SilkS) (width 0.15))
-    (pad 1 thru_hole circle (at 0 0) (size 3.375 3.375) (drill 2.325) (layers *.Cu *.Mask F.SilkS))
   )
   (module altimeterComponentFootprints:6-UFDFN_Exposed_Pad (layer F.Cu)
@@
     (pad 2 smd rect (at 1.25 0 90) (size 1 1.8) (layers F.Cu F.Paste F.Mask)
       (net 5 "Net-(C3-Pad3)"))
+  )
+  (gr_text v0.1 (at 170.4 53) (layer F.SilkS)
+    (effects (font (size 2 2) (thickness 0.5)))
   )
   (gr_line (start 127 50.8) (end 127 69.85) (angle 90) (layer Edge.Cuts) (width 0.15))
@@
   (segment (start 143.8291 65.8458) (end 144.8615 64.8134) (width 0.2032) (layer F.Cu) (net 38))
   (segment (start 143.4498 65.8458) (end 143.8291 65.8458) (width 0.2032) (layer F.Cu) (net 38))
+  (zone (net 1) (net_name GND) (layer F.Cu) (hatch edge 0.508)
+    (connect_pads (clearance 0.1524))
+    (min_thickness 0.1524)
+    (fill yes (arc_segments 16) (thermal_gap 0.508) (thermal_bridge_width 0.508))
+    (polygon
+      (pts
+        (xy 127 50.8) (xy 177.8 50.85) (xy 177.75 69.9) (xy 126.95 69.85)
+      )
+    )
+  )
+  (zone (net 1) (net_name GND) (layer B.Cu) (hatch edge 0.508)
+    (connect_pads (clearance 0.1524))
+    (min_thickness 0.1524)
+    (fill yes (arc_segments 16) (thermal_gap 0.508) (thermal_bridge_width 0.508))
+    (polygon
+      (pts
+        (xy 127 50.8) (xy 177.8 50.8) (xy 177.85 69.85) (xy 127.05 69.8)
+      )
+    )
+  )
 )

Commit message: Sod Blaster Tri Cities 2019 - clean code, hardware
Routing:
- removed copper zone on B.Cu, net GND
- removed copper zone on F.Cu, net GND
Other:
- rule pad_to_mask_clearance: 0.2 -> 0.0508
- board text added: "+"
- board text added: "-"
- board text added: "3RD"
- board text added: "APO"
- board text added: "MAIN"
Changed lines of the file:
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@@
     (links 145)
     (no_connects 0)
-    (area 126.1718 47.556257 178.6038 77.258)
+    (area 124.313467 47.556257 178.6038 77.258)
     (thickness 1.6)
-    (drawings 5)
+    (drawings 10)
     (tracks 840)
     (zones 0)
@@
     (pad_size 1.524 1.524)
     (pad_drill 0.762)
-    (pad_to_mask_clearance 0.2)
+    (pad_to_mask_clearance 0.0508)
     (aux_axis_origin 0 0)
     (visible_elements 7FFEFFFF)
@@
   (module altimeterComponentFootprints:C_array_2x_0805 (layer F.Cu)
     (at 158.6 52.5 270)
-    (fp_text reference C1 (at 0.05 -1.5 270) (layer F.SilkS)
+    (fp_text reference C1 (at 0.6 -1.45 270) (layer F.SilkS)
       (effects (font (size 0.75 0.75) (thickness 0.15)))
     )
@@
     (tags "capacitor 0603")
     (attr smd)
-    (fp_text reference C4 (at 1.95 0.25 360) (layer F.SilkS)
-      (effects (font (size 1 1) (thickness 0.15)))
+    (fp_text reference C4 (at 1.9 0.05 360) (layer F.SilkS)
+      (effects (font (size 0.75 0.75) (thickness 0.15)))
     )
     (fp_text value 0.1uF (at 0 1.5 270) (layer F.Fab)
@@
     (tags "capacitor 0603")
     (attr smd)
-    (fp_text reference C5 (at 2.2 0 90) (layer F.SilkS)
+    (fp_text reference C5 (at 2.2 0 180) (layer F.SilkS)
       (effects (font (size 1 1) (thickness 0.15)))
     )
@@
     (tags "capacitor 0603")
     (attr smd)
-    (fp_text reference C9 (at 2.2 -0.05 90) (layer F.SilkS)
+    (fp_text reference C9 (at 2.05 -0.05 270) (layer F.SilkS)
       (effects (font (size 1 1) (thickness 0.15)))
     )
@@
     (tags "capacitor 0603")
     (attr smd)
-    (fp_text reference C13 (at 2.1 -2.45 360) (layer F.SilkS)
-      (effects (font (size 1 1) (thickness 0.15)))
+    (fp_text reference C13 (at 2.1 0.4 360) (layer F.SilkS)
+      (effects (font (size 0.75 0.75) (thickness 0.15)))
     )
     (fp_text value 0.1uF (at 0 1.5 270) (layer F.Fab)
@@
     (tags "capacitor 0603")
     (attr smd)
-    (fp_text reference C17 (at -2.1 -2.5 180) (layer F.SilkS)
-      (effects (font (size 1 1) (thickness 0.15)))
+    (fp_text reference C17 (at -2.05 0.5 180) (layer F.SilkS)
+      (effects (font (size 0.75 0.75) (thickness 0.15)))
     )
     (fp_text value 0.1uF (at 0 1.5 90) (layer F.Fab)
@@
     (tags "capacitor 0603")
     (attr smd)
-    (fp_text reference L1 (at -1.75 0.05 180) (layer F.SilkS)
-      (effects (font (size 1 1) (thickness 0.15)))
+    (fp_text reference L1 (at -1.85 0.05 180) (layer F.SilkS)
+      (effects (font (size 0.75 0.75) (thickness 0.15)))
     )
     (fp_text value 10uH (at 0 1.5 90) (layer F.Fab)
@@
   (module altimeterComponentFootprints:R_array_4x_1206 (layer F.Cu)
     (at 174.95 67.25 270)
-    (fp_text reference R1 (at -2.35 0 360) (layer F.SilkS)
+    (fp_text reference R1 (at -2.1 -0.05 540) (layer F.SilkS)
       (effects (font (size 0.75 0.75) (thickness 0.15)))
     )
@@
   (module altimeterComponentFootprints:R_array_4x_1206 (layer F.Cu)
     (at 166.15 67.3 90)
-    (fp_text reference R2 (at -1 -2 90) (layer F.SilkS)
+    (fp_text reference R2 (at 2.1 0.7 180) (layer F.SilkS)
       (effects (font (size 0.75 0.75) (thickness 0.15)))
     )
@@
   (module altimeterComponentFootprints:R_array_4x_1206 (layer F.Cu)
     (at 171 67.25 90)
-    (fp_text reference R3 (at -1 -2.05 90) (layer F.SilkS)
+    (fp_text reference R3 (at 2.1 0 180) (layer F.SilkS)
       (effects (font (size 0.75 0.75) (thickness 0.15)))
     )
@@
     (tags "resistor 0603")
     (attr smd)
-    (fp_text reference R4 (at 2.05 0 90) (layer F.SilkS)
+    (fp_text reference R4 (at 2.05 0 180) (layer F.SilkS)
       (effects (font (size 1 1) (thickness 0.15)))
     )
@@
   (module altimeterComponentFootprints:R_1206 (layer F.Cu)
     (at 162.15 63.7)
-    (fp_text reference R5 (at 3.7 0.95 90) (layer F.SilkS)
+    (fp_text reference R5 (at 0.75 2.15 180) (layer F.SilkS)
       (effects (font (size 1 1) (thickness 0.15)) (justify left bottom))
     )
@@
   (module altimeterComponentFootprints:R_array_4x_1206 (layer F.Cu)
     (at 150.5 53.15 270)
-    (fp_text reference R6 (at -1 -2 270) (layer F.SilkS)
+    (fp_text reference R6 (at 2.35 -0.95 360) (layer F.SilkS)
       (effects (font (size 0.75 0.75) (thickness 0.15)))
     )
@@
       (effects (font (size 0.84455 0.84455) (thickness 0.09779)) (justify left bottom))
     )
-    (fp_text value H3LIS331DL (at -1.905 0.635 90) (layer F.SilkS)
+    (fp_text value H3LIS331DL (at -1.6 0.2 90) (layer Eco2.User)
       (effects (font (size 0.60325 0.60325) (thickness 0.0635)) (justify left bottom))
     )
@@
     (pad 2 smd rect (at 1.25 0 90) (size 1 1.8) (layers F.Cu F.Paste F.Mask)
       (net 5 "Net-(C3-Pad3)"))
+  )
+  (gr_text 3RD (at 173.45 68.15) (layer B.SilkS)
+    (effects (font (size 1.2 1.2) (thickness 0.3)) (justify mirror))
+  )
+  (gr_text APO (at 168.4 68.15) (layer B.SilkS)
+    (effects (font (size 1.2 1.2) (thickness 0.3)) (justify mirror))
+  )
+  (gr_text MAIN (at 173.45 51.6 180) (layer B.SilkS)
+    (effects (font (size 1.2 1.2) (thickness 0.3)) (justify mirror))
+  )
+  (gr_text - (at 167.05 51.65) (layer B.SilkS)
+    (effects (font (size 1.5 1.5) (thickness 0.3)) (justify mirror))
+  )
+  (gr_text + (at 169.55 51.65) (layer B.SilkS)
+    (effects (font (size 1.5 1.5) (thickness 0.3)) (justify mirror))
   )
   (gr_text v0.1 (at 170.4 53) (layer F.SilkS)
@@
   (segment (start 143.8291 65.8458) (end 144.8615 64.8134) (width 0.2032) (layer F.Cu) (net 38))
   (segment (start 143.4498 65.8458) (end 143.8291 65.8458) (width 0.2032) (layer F.Cu) (net 38))
-  (zone (net 1) (net_name GND) (layer F.Cu) (hatch edge 0.508)
-    (connect_pads (clearance 0.1524))
-    (min_thickness 0.1524)
-    (fill yes (arc_segments 16) (thermal_gap 0.508) (thermal_bridge_width 0.508))
-    (polygon
-      (pts
-        (xy 127 50.8) (xy 177.8 50.85) (xy 177.75 69.9) (xy 126.95 69.85)
-      )
-    )
-  )
-  (zone (net 1) (net_name GND) (layer B.Cu) (hatch edge 0.508)
-    (connect_pads (clearance 0.1524))
-    (min_thickness 0.1524)
-    (fill yes (arc_segments 16) (thermal_gap 0.508) (thermal_bridge_width 0.508))
-    (polygon
-      (pts
-        (xy 127 50.8) (xy 177.8 50.8) (xy 177.85 69.85) (xy 127.05 69.8)
-      )
-    )
-  )
 )
